File: project_files/project_files.kicad_sch (KiCad schematic)
At the start: 27 parts, among them SW11 SW_Push, SW12 SW_Push, SW13 SW_Push, SW17 SW_Push, SW18 SW_Push, SW19 SW_Push, SW3 SW_Push, SW4 SW_Push, SW5 SW_Push, SW7 SW_Push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

Commit message: test pads
no more castellated holes
my wallet is saved
Parts:
- added 1L1, 1R1, 2L1, 2R1, 3L1, 3R1, 7L1, 7R1, 8L1, 8R1, 9L1, 9R1: TestPoint, TestPoint:TestPoint_Pad_D1.0mm, symbol Connector:TestPoint
Connections:
- net PIN_1: now also 1L1.1, 1R1.1
- net PIN_2: now also 2L1.1, 2R1.1
- net PIN_3: now also 3L1.1, 3R1.1
- net PIN_7: now also 7L1.1, 7R1.1
- net PIN_8: now also 8L1.1, 8R1.1
- net PIN_9: now also 9L1.1, 9R1.1
