File: project_files/after_soldering.kicad_pcb (KiCad board)
At the start: 2 copper layers, 95.3 x 104.8 mm, 48 parts, among them SW11 SW_Push, SW12 SW_Push, SW13 SW_Push, SW17 SW_Push, SW18 SW_Push, SW19 SW_Push, SW3 SW_Push, SW4 SW_Push, SW5 SW_Push, SW7 SW_Push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

Commit message: after solder
and curves :)
Parts:
- removed the REF** at (175.2, 90.5)
- removed the REF** at (128.4, 90.5)
- removed the REF** at (137.8, 90.5)
- removed the REF** at (119.1, 90.5)
- removed the REF** at (180.3, 90.5)
- removed the REF** at (165.8, 90.5)
- removed the REF** at (156.5, 90.5)
- removed the REF** at (147.1, 90.5)
- added REF**: BreakLine_11h_D0.5mm_P0.85mm, Panelization:BreakLine_11h_D0.5mm_P0.85mm, F.Cu at (190.5, 121.8)
- moved 3R1 58.8 mm to (155.8, 102.3)
- moved 7R1 58.8 mm to (146.3, 88.4)
- moved D14 58.8 mm to (158.4, 88.4)
- moved D15 58.8 mm to (177.6, 88.4)
- moved D21 58.8 mm to (187.1, 117.0)
- moved SW17 58.8 mm to (176.2, 73.8)
- moved SW19 58.8 mm to (185.8, 102.3)
- moved 1R1 58.8 mm to (146.3, 95.6)
- moved 2R1 58.8 mm to (146.3, 92.0)
- moved 8R1 58.8 mm to (155.8, 117.0)
- moved 9R1 58.8 mm to (155.8, 119.4)
- moved D20 58.8 mm to (168.0, 117.0)
- moved OLED1 58.8 mm to (229.2, 76.5)
- moved SW11 58.8 mm to (157.2, 73.8)
- moved SW13 58.8 mm to (166.8, 102.3)
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Other:
- board size 95.3 x 104.8 mm -> 181 x 52.4 mm

Commit message: oled centered
with silkscreen!
Parts:
- moved 1R1 173.6 mm to (-8.33, 16.7)
- moved 2L1 173.6 mm to (-10.7, 13.1)
- moved 2R1 173.6 mm to (-8.33, 13.1)
- moved 3L1 173.6 mm to (-1.19, 23.5)
- moved 3R1 173.6 mm to (1.20, 23.5)
- moved 7L1 173.6 mm to (-10.7, 9.53)
- moved 7R1 173.6 mm to (-8.33, 9.53)
- moved 8L1 173.6 mm to (-1.19, 38.1)
- moved 8R1 173.6 mm to (1.20, 38.1)
- moved 9L1 173.6 mm to (-1.19, 40.5)
- moved 9R1 173.6 mm to (1.20, 40.5)
- moved D13 173.6 mm to (-15.2, 9.53)
- moved D14 173.6 mm to (3.81, 9.53)
- moved D15 173.6 mm to (22.9, 9.53)
- moved D16 173.6 mm to (-81.9, 38.1)
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
Commit message: lots of case work
pcb subject to change, so no gerbers yet
Parts:
- removed REF** (x2): BreakLine_11h_D0.5mm_P0.85mm, Panelization:BreakLine_11h_D0.5mm_P0.85mm
- SW11, SW12, SW13, SW17, SW18, SW19, SW3, SW4, SW5, SW7, SW8, SW9: footprint Button_Switch_Keyboard:SW_Cherry_MX_1.00u_PCB -> custom:SW_Cherry_MX_1.00u_PCB
- SongSelect1: footprint Rotary_Encoder:RotaryEncoder_Alps_EC11E-Switch_Vertical_H20mm -> custom:RotaryEncoder_Alps_EC11E-Switch_Vertical_H20mm
- moved OLED1 198.7 mm to (255.4, 80.9)
- moved 3L1 197.8 mm to (179.6, 103.5)
- moved 8L1 197.8 mm to (179.6, 118.2)
- moved 9L1 197.8 mm to (179.6, 120.6)
- moved D16 197.8 mm to (98.9, 118.2)
- moved D18 197.8 mm to (137.0, 118.2)
- moved SW12 197.8 mm to (116.7, 103.6)
- moved SongSelect1 197.8 mm to (230.9, 82.6)
- moved 1L1 197.8 mm to (170.1, 96.8)
- moved 1R1 197.8 mm to (172.5, 96.8)
- moved 2L1 197.8 mm to (170.1, 93.2)
- moved 2R1 197.8 mm to (172.5, 93.2)
- moved 3R1 197.8 mm to (182.0, 103.5)
- moved 7L1 197.8 mm to (170.1, 89.6)
- moved 7R1 197.8 mm to (172.5, 89.6)
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Routing:
- net /SCL: track 30.8 -> 34.0 mm
- net /SDA: track 34.4 -> 37.6 mm
- net /PWR_3v3: track 66.8 -> 70.0 mm
- net GND: track 77.5 -> 80.7 mm
Other:
- outline, holes or cut-outs redrawn
